File: motor-control/driver.sch (KiCad schematic (older format))
At the start: 25 parts, among them U4 DRV8301

Commit message: Added values in schematic, new diode&induct ftpnts
Parts:
- L1: footprint p16261:inductor_custom -> p16261:PHC-27-683
Changed lines of the file:
@@
 F 0 "L1" H 6480 2490 50  0000 L CNN
 F 1 "68uH" H 6480 2410 50  0000 L CNN
-F 2 "p16261:inductor_custom" H 6450 2450 60  0001 C CNN
+F 2 "p16261:PHC-27-683" H 6450 2450 60  0001 C CNN
 F 3 "http://www.coilcraft.com/pdfs/pch.pdf" H 6450 2450 60  0001 C CNN
 	1    6450 2450

Commit message: rid bad 3d, add new cap thruhole, add datasht lnks
Parts:
- C18: footprint Capacitors_SMD:C_0805 -> p16261:FK20X7S2A475K
- R27: footprint Resistors_SMD:R_0805 -> Resistors_SMD:R_0603
Changed lines of the file:
@@
 LIBS:contrib
 LIBS:valves
+LIBS:p16261
+LIBS:my_lib
 LIBS:_saved_motor-control-cache
 EELAYER 25 0
@@
 F 0 "C18" H 6775 2000 50  0000 L CNN
 F 1 "10uF" H 6775 1800 50  0000 L CNN
-F 2 "Capacitors_SMD:C_0805" H 6788 1750 30  0001 C CNN
-F 3 "" H 6750 1900 60  0000 C CNN
+F 2 "p16261:FK20X7S2A475K" H 6788 1750 30  0001 C CNN
+F 3 "http://www.mouser.com/ProductDetail/TDK/FK20X7S2A475K/?qs=sGAEpiMZZMt3KoXD5rJ2N48tYEMqcp4xHF5PfUWuJkY%3d" H 6750 1900 60  0001 C CNN
 F 4 "100 V" H 6750 1900 60  0001 C CNN "Voltage"
 	1    6750 1900
@@
 F 1 "10pF" H 2260 2170 50  0000 L CNN
 F 2 "Capacitors_SMD:C_0805" H 2250 2250 60  0001 C CNN
-F 3 "" H 2250 2250 60  0000 C CNN
+F 3 "http://www.mouser.com/ProductDetail/AVX/04025A100FAT2A/?qs=sGAEpiMZZMsh%252b1woXyUXj6IVtf51%2fGgBI68mQP5hS%252bo%3d" H 2250 2250 60  0001 C CNN
 	1    2250 2250
 	1    0    0    -1
@@
 F 1 "0.01uF" H 2710 2070 50  0000 L CNN
 F 2 "Capacitors_SMD:C_0805" H 2700 2150 60  0001 C CNN
-F 3 "" H 2700 2150 60  0000 C CNN
+F 3 "http://www.mouser.com/Search/ProductDetail.aspx?R=CC0805KRX7R9BB103virtualkey60120000virtualkey603-CC805KRX7R9BB103" H 2700 2150 60  0001 C CNN
 	1    2700 2150
 	1    0    0    -1
@@
 F 0 "R27" V 3980 1950 50  0000 C CNN
 F 1 "205k" V 3900 1950 50  0000 C CNN
-F 2 "Resistors_SMD:R_0805" V 3830 1950 30  0001 C CNN
-F 3 "" H 3900 1950 30  0000 C CNN
+F 2 "Resistors_SMD:R_0603" V 3830 1950 30  0001 C CNN
+F 3 "http://www.mouser.com/Search/ProductDetail.aspx?R=TNPW0603205KBEEAvirtualkey61300000virtualkey71-TNPW0603205KBEEA" H 3900 1950 30  0001 C CNN
 	1    3900 1950
 	0    1    1    0
@@
 F 1 "1uF" H 3510 4070 50  0000 L CNN
 F 2 "Capacitors_SMD:C_0805" H 3500 4150 60  0001 C CNN
-F 3 "" H 3500 4150 60  0000 C CNN
+F 3 "http://www.mouser.com/ProductDetail/TDK/C2012X7S2A105K125AB/?qs=sGAEpiMZZMsh%252b1woXyUXj0VscQlT5uEB2auVtHOVuSQ%3d" H 3500 4150 60  0001 C CNN
 F 4 "6.3 V" H 3500 4150 60  0001 C CNN "Voltage"
 	1    3500 4150
@@
 F 1 "1uF" H 3610 4470 50  0000 L CNN
 F 2 "Capacitors_SMD:C_0805" H 3600 4550 60  0001 C CNN
-F 3 "" H 3600 4550 60  0000 C CNN
+F 3 "http://www.mouser.com/ProductDetail/TDK/C2012X7S2A105K125AB/?qs=sGAEpiMZZMsh%252b1woXyUXj0VscQlT5uEB2auVtHOVuSQ%3d" H 3600 4550 60  0001 C CNN
 F 4 "10 V" H 3600 4550 60  0001 C CNN "Voltage"
 	1    3600 4550
@@
 F 1 "10k" V 3100 2400 50  0000 C CNN
 F 2 "Resistors_SMD:R_0805" V 3030 2400 30  0001 C CNN
-F 3 "" H 3100 2400 30  0000 C CNN
+F 3 "http://www.mouser.com/Search/ProductDetail.aspx?R=CRCW080510K0FKEAvirtualkey61300000virtualkey71-CRCW0805-10K-E3" H 3100 2400 30  0001 C CNN
 	1    3100 2400
 	1    0    0    -1
@@
 F 1 "10k" V 3300 2400 50  0000 C CNN
 F 2 "Resistors_SMD:R_0805" V 3230 2400 30  0001 C CNN
-F 3 "" H 3300 2400 30  0000 C CNN
+F 3 "http://www.mouser.com/Search/ProductDetail.aspx?R=CRCW080510K0FKEAvirtualkey61300000virtualkey71-CRCW0805-10K-E3" H 3300 2400 30  0001 C CNN
 	1    3300 2400
 	1    0    0    -1
@@
 F 1 "0R" V 3900 2550 50  0000 C CNN
 F 2 "Resistors_SMD:R_0805" V 3830 2550 30  0001 C CNN
-F 3 "" H 3900 2550 30  0000 C CNN
+F 3 "http://www.mouser.com/ProductDetail/Panasonic/ERJ-6GEY0R00V/?qs=sGAEpiMZZMtlubZbdhIBIGGkozl1QdRpbM2mlUXXIDw%3d" H 3900 2550 30  0001 C CNN
 	1    3900 2550
 	0    1    1    0
@@
 F 1 "0.022uF" H 3810 3220 50  0000 L CNN
 F 2 "Capacitors_SMD:C_0805" H 3800 3300 60  0001 C CNN
-F 3 "" H 3800 3300 60  0000 C CNN
+F 3 "http://www.mouser.com/Search/ProductDetail.aspx?R=C2012X7R2E223K125AAvirtualkey52130000virtualkey810-C2012X7R2E223K" H 3800 3300 60  0001 C CNN
 	1    3800 3300
 	1    0    0    -1
@@
 F 1 "1uF" H 5710 4720 50  0000 L CNN
 F 2 "Capacitors_SMD:C_0805" H 5700 4800 50  0001 C CNN
-F 3 "" H 5700 4800 50  0000 C CNN
+F 3 "http://www.mouser.com/ProductDetail/TDK/C2012X7S2A105K125AB/?qs=sGAEpiMZZMsh%252b1woXyUXj0VscQlT5uEB2auVtHOVuSQ%3d" H 5700 4800 50  0001 C CNN
 F 4 "100 V" H 5700 4800 60  0001 C CNN "Voltage"
 	1    5700 4800
